Commit message: Rerecord the TIAGo + Stretch warehouse demo with every step parameter
warehouse_tiago_stretch_totes (203.3 s) is recorded again from
WarehouseTwin d5c8b34 with cramera's viewer/readable-step-cards (080fa36):
each plan step now carries every parameter it ran with (object, arm, grasp,
rail height, target poses), the totes are named by their name and goods
("A08 · computer mouse box") instead of their body UUID, and the robot is
named "stretch" instead of "stretch_<identity>", in index.json too.
Placement: A08 7.1 mm, A09 9.6 mm, R01 1.0 mm. The bundle passes
cramera-check-bundle.

Co-Authored-By: Claude Opus 5.5 <noreply@anthropic.com>

File: warehouse_tiago_stretch_totes/environment.urdf (robot description, URDF)
Before this commit: robot environment, 719 links, 718 joints
Links:
- removed link 6404d406-4935-4ad1-8639-137749d23c8c/odom
- removed link e352aac8-5b24-4d7e-9bf5-365512cf710b/odom
- added link b0140898-e215-495d-b5ed-96815bdb0d90/odom
- added link fddcc0dc-77fe-4358-8424-d76119505e90/odom
Joints:
- removed joint 6404d406-4935-4ad1-8639-137749d23c8c/map_T_odom
- removed joint e352aac8-5b24-4d7e-9bf5-365512cf710b/map_T_odom
- added joint b0140898-e215-495d-b5ed-96815bdb0d90/map_T_odom: type floating, parent map, child b0140898-e215-495d-b5ed-96815bdb0d90/odom, origin xyz=0.0 0.0 0.0 rpy=0.0 0.0 0.0
- added joint fddcc0dc-77fe-4358-8424-d76119505e90/map_T_odom: type floating, parent map, child fddcc0dc-77fe-4358-8424-d76119505e90/odom, origin xyz=0.0 0.0 0.0 rpy=0.0 0.0 0.0

File: warehouse_tiago_stretch_totes/stretch_6679361b8bfc4e76b861deb96ed1f4cc.urdf (robot description, URDF)
Before this commit: robot stretch_04284f6532c945f098f6ac3ea2eeda6e, 47 links, 46 joints
Joints:
- joint stretch_description/camera_accel_optical_joint: origin xyz=0.0 0.0 0.0 rpy=-1.570796 0.0 -1.570796 -> xyz=-0.0 0.0 0.0 rpy=-1.570796 0.0 -1.570796
- joint stretch_description/camera_gyro_optical_joint: origin xyz=0.0 0.0 0.0 rpy=-1.570796 0.0 -1.570796 -> xyz=-0.0 0.0 0.0 rpy=-1.570796 0.0 -1.570796
- joint stretch_description/joint_arm_l4: origin xyz=-0.2547 0.0 0.0 rpy=1.5708 0.0 -1.5708 -> xyz=-0.2547 0.0 -0.0 rpy=1.5708 0.0 -1.5708
- joint stretch_description/joint_head: origin xyz=-0.0 1.33 0.0 rpy=-1.570789 -1.570796 0.0 -> xyz=0.0 1.33 -0.0 rpy=-1.570789 -1.570796 0.0

File: warehouse_tiago_stretch_totes/tiago_bf1eeb1d694f4cca964143141cbc066d.urdf (robot description, URDF)
Before this commit: robot tiago_01f0629227a64bd3891e1bf7c58230dc, 103 links, 102 joints
Joints:
- joint tiago_dual/base_dock: origin xyz=0.2675 -0.0 0.061 rpy=0.0 0.0 0.0 -> xyz=0.2675 0.0 0.061 rpy=0.0 0.0 0.0
- joint tiago_dual/base_footprint_joint: origin xyz=0.0 -0.0 0.0985 rpy=0.0 0.0 0.0 -> xyz=0.0 0.0 0.0985 rpy=0.0 0.0 0.0
- joint tiago_dual/base_imu_joint: origin xyz=0.10171 -0.0 0.11282 rpy=0.0 0.0 -1.570796 -> xyz=0.10171 0.0 0.11282 rpy=0.0 0.0 -1.570796
- joint tiago_dual/base_laser_joint: origin xyz=0.202 -0.0 -0.004 rpy=0.0 0.0 0.0 -> xyz=0.202 0.0 -0.004 rpy=0.0 0.0 0.0
- joint tiago_dual/base_sonar_02_joint: origin xyz=-0.259 -0.0 0.173 rpy=0.0 0.0 3.141593 -> xyz=-0.259 0.0 0.173 rpy=0.0 0.0 3.141593
- joint tiago_dual/caster_back_left_2_joint: origin xyz=-0.016 -0.0 -0.04 rpy=-1.570796 0.0 0.0 -> xyz=-0.016 0.0 -0.04 rpy=-1.570796 0.0 0.0
- joint tiago_dual/caster_back_right_2_joint: origin xyz=-0.016 -0.0 -0.04 rpy=-1.570796 0.0 0.0 -> xyz=-0.016 0.0 -0.04 rpy=-1.570796 0.0 0.0
- joint tiago_dual/cover_joint: origin xyz=0.0 -0.0 0.13 rpy=0.0 0.0 0.0 -> xyz=0.0 0.0 0.13 rpy=0.0 0.0 0.0
- joint tiago_dual/gripper_left_base_joint: origin xyz=-0.0 0.0 0.0312 rpy=0.0 0.0 0.0 -> xyz=0.0 0.0 0.0312 rpy=0.0 0.0 0.0
- joint tiago_dual/gripper_left_coupler_joint: origin xyz=0.0 0.0 0.0 rpy=1.570796 0.0 1.570796 -> xyz=-0.0 -0.0 0.0 rpy=1.570796 0.0 1.570796
- joint tiago_dual/gripper_left_left_outer_finger_joint: origin xyz=0.0 0.0315 -0.0041 rpy=0.0 0.0 0.0 -> xyz=-0.0 0.0315 -0.0041 rpy=0.0 0.0 0.0
- joint tiago_dual/gripper_left_right_inner_finger_pad_joint: origin xyz=0.0 -0.02202 0.03242 rpy=0.0 0.0 0.0 -> xyz=-0.0 -0.02202 0.03242 rpy=0.0 0.0 0.0
- joint tiago_dual/gripper_right_base_joint: origin xyz=-0.0 0.0 0.0312 rpy=0.0 0.0 0.0 -> xyz=-0.0 -0.0 0.0312 rpy=0.0 0.0 0.0
- joint tiago_dual/gripper_right_coupler_joint: origin xyz=0.0 0.0 0.0 rpy=1.570796 0.0 1.570796 -> xyz=0.0 0.0 -0.0 rpy=1.570796 -0.0 1.570796
- joint tiago_dual/gripper_right_grasping_frame_Y_joint: origin xyz=0.0 0.0 0.11 rpy=1.5708 0.0 0.0 -> xyz=-0.0 0.0 0.11 rpy=1.5708 0.0 0.0
- joint tiago_dual/gripper_right_grasping_frame_Z_joint: origin xyz=0.0 0.0 0.11 rpy=0.0 0.0 0.0 -> xyz=-0.0 0.0 0.11 rpy=0.0 0.0 0.0
- joint tiago_dual/gripper_right_grasping_frame_joint: origin xyz=0.0 0.0 0.11 rpy=-3.141593 -1.570793 3.141593 -> xyz=-0.0 0.0 0.11 rpy=3.141593 -1.570793 -3.141593
- joint tiago_dual/gripper_right_left_inner_finger_joint_mimic: origin xyz=0.0 0.0 0.0 rpy=0.0 0.0 0.0 -> xyz=-0.0 -0.0 0.0 rpy=0.0 0.0 0.0
- joint tiago_dual/gripper_right_left_inner_finger_pad_joint: origin xyz=-0.0 -0.02202 0.03242 rpy=0.0 0.0 0.0 -> xyz=0.0 -0.02202 0.03242 rpy=0.0 0.0 0.0
- joint tiago_dual/gripper_right_left_inner_finger_pad_joint_mimic: origin xyz=0.0 0.0 0.0 rpy=0.0 0.0 0.0 -> xyz=-0.0 -0.0 0.0 rpy=0.0 0.0 0.0
- joint tiago_dual/gripper_right_left_inner_knuckle_joint_mimic: origin xyz=0.0 0.0 0.0 rpy=0.0 0.0 0.0 -> xyz=-0.0 -0.0 0.0 rpy=0.0 0.0 0.0
- joint tiago_dual/gripper_right_left_outer_finger_joint_mimic: origin xyz=0.0 0.0 0.0 rpy=0.0 0.0 0.0 -> xyz=-0.0 -0.0 0.0 rpy=0.0 0.0 0.0
- joint tiago_dual/gripper_right_right_inner_finger_joint_mimic: origin xyz=0.0 0.0 0.0 rpy=0.0 0.0 0.0 -> xyz=-0.0 -0.0 0.0 rpy=0.0 0.0 0.0
- joint tiago_dual/gripper_right_right_inner_finger_pad_joint_mimic: origin xyz=0.0 0.0 0.0 rpy=0.0 0.0 0.0 -> xyz=-0.0 -0.0 0.0 rpy=0.0 0.0 0.0
- joint tiago_dual/gripper_right_right_inner_knuckle_joint_mimic: origin xyz=0.0 0.0 0.0 rpy=0.0 0.0 0.0 -> xyz=-0.0 -0.0 0.0 rpy=0.0 0.0 0.0
- joint tiago_dual/gripper_right_right_outer_finger_joint_mimic: origin xyz=0.0 0.0 0.0 rpy=0.0 0.0 0.0 -> xyz=-0.0 -0.0 0.0 rpy=0.0 0.0 0.0
- joint tiago_dual/gripper_right_right_outer_knuckle_joint_mimic: origin xyz=0.0 0.0 0.0 rpy=0.0 0.0 0.0 -> xyz=-0.0 -0.0 0.0 rpy=0.0 0.0 0.0
- joint tiago_dual/head_front_camera_color_joint: origin xyz=-0.0 0.022 0.0 rpy=0.0 0.0 0.0 -> xyz=0.0 0.022 0.0 rpy=0.0 0.0 0.0
- joint tiago_dual/head_front_camera_color_optical_joint: origin xyz=-0.0 0.0 0.0 rpy=-1.570796 0.0 -1.570796 -> xyz=0.0 0.0 0.0 rpy=-1.570796 0.0 -1.570796
- joint tiago_dual/head_front_camera_depth_optical_joint: origin xyz=0.0 -0.0 0.0 rpy=-1.570796 0.0 -1.570796 -> xyz=0.0 0.0 0.0 rpy=-1.570796 0.0 -1.570796
- joint tiago_dual/head_front_camera_optical_joint: origin xyz=0.0 0.0 0.0 rpy=-1.570796 0.0 -1.570796 -> xyz=-0.0 0.0 0.0 rpy=-1.570796 0.0 -1.570796
- joint tiago_dual/suspension_left_joint: origin xyz=0.0 -0.0 0.0 rpy=0.0 0.0 0.0 -> xyz=0.0 0.0 0.0 rpy=0.0 0.0 0.0
- joint tiago_dual/suspension_right_joint: origin xyz=0.0 -0.0 0.0 rpy=0.0 0.0 0.0 -> xyz=0.0 0.0 0.0 rpy=0.0 0.0 0.0
